Commit message: added 2D LiDAR & changed some model colours

File: model/vehicle.xacro (robot description, xacro)
@@ -1,4 +1,5 @@
 <?xml version="1.0"?>
 <robot name="ackermann_steering_vehicle" xmlns:xacro="http://www.ros.org/wiki/xacro">
+  <xacro:include filename="inertial_macros.xacro"/>
   <!-- Arguments -->
   <xacro:arg name="body_length" default="2.0" />
@@ -14,12 +15,4 @@
   <xacro:arg name="max_velocity" default="1.0" />
   <xacro:arg name="max_effort" default="10.0" />
-  <xacro:arg name="camera_box_size" default="0.1" />
-  <xacro:arg name="camera_stick_size" default="0.2" />
-  <xacro:arg name="camera_height" default="1.5" />
-  <xacro:arg name="camera_pitch" default="0.1" />
-  <xacro:arg name="camera_fov" default="1.396263" />
-  <xacro:arg name="camera_fps" default="30" />
-  <xacro:arg name="image_width" default="640" />
-  <xacro:arg name="image_height" default="480" />
   <!-- Mathematical Constants -->
   <xacro:property name="PI" value="3.14159265"/>
@@ -37,12 +30,4 @@
   <xacro:property name="max_velocity" value="$(arg max_velocity)"/>
   <xacro:property name="max_effort" value="$(arg max_effort)"/>
-  <xacro:property name="camera_box_size" value="$(arg camera_box_size)"/>
-  <xacro:property name="camera_stick_size" value="$(arg camera_stick_size)"/>
-  <xacro:property name="camera_height" value="$(arg camera_height)"/>
-  <xacro:property name="camera_pitch" value="$(arg camera_pitch)"/>
-  <xacro:property name="camera_fov" value="$(arg camera_fov)"/>
-  <xacro:property name="camera_fps" value="$(arg camera_fps)"/>
-  <xacro:property name="image_width" value="$(arg image_width)"/>
-  <xacro:property name="image_height" value="$(arg image_height)"/>
   <xacro:property name="body_mass" value="${body_density * body_length * body_height * body_width}"/>
   <xacro:property name="body_inertia_x" value="${1.0/12.0 * body_mass * (body_height*body_height + body_width*body_width)}"/>
@@ -60,5 +45,5 @@
   <link name="body_link">
     <visual>
-      <origin xyz="0.0 0.0 0.0" rpy="0.0 0.0 0.0"/>
+      <origin xyz="0.0 0.0 ${body_height/2}" rpy="0.0 0.0 0.0"/>
       <geometry>
         <box size="${body_length} ${body_width} ${body_height}"/>
@@ -69,5 +54,5 @@
     </visual>
     <collision>
-      <origin xyz="0.0 0.0 0.0" rpy="0.0 0.0 0.0"/>
+      <origin xyz="0.0 0.0 ${body_height/2}" rpy="0.0 0.0 0.0"/>
       <geometry>
         <box size="${body_length} ${body_width} ${body_height}"/>
@@ -77,5 +62,5 @@
       <mass value="${body_mass}"/>
       <inertia ixx="${body_inertia_x}" ixy="0.0" ixz="0.0" iyy="${body_inertia_y}" iyz="0" izz="${body_inertia_z}"/>
-      <origin xyz="0 0 0" rpy="0 0 0"/>
+      <origin xyz="0 0 ${body_height/2}" rpy="0 0 0"/>
     </inertial>
   </link>
@@ -88,5 +73,5 @@
       </geometry>
       <material name="wheel_material">
-        <color rgba="0.0 0.0 0.0 1.0"/>
+        <color rgba="1.0 0.91 0.09 1.0"/>
       </material>
     </visual>
@@ -111,5 +96,5 @@
       </geometry>
       <material name="wheel_material">
-        <color rgba="0.0 0.0 0.0 1.0"/>
+        <color rgba="1.0 0.91 0.09 1.0"/>
       </material>
     </visual>
@@ -134,5 +119,5 @@
       </geometry>
       <material name="wheel_material">
-        <color rgba="0.0 0.0 0.0 1.0"/>
+        <color rgba="1.0 0.91 0.09 1.0"/>
       </material>
     </visual>
@@ -157,5 +142,5 @@
       </geometry>
       <material name="wheel_material">
-        <color rgba="0.0 0.0 0.0 1.0"/>
+        <color rgba="1.0 0.91 0.09 1.0"/>
       </material>
     </visual>
@@ -180,5 +165,5 @@
       </geometry>
       <material name="wheel_material">
-        <color rgba="0.0 0.0 0.0 1.0"/>
+        <color rgba="1.0 0.91 0.09 1.0"/>
       </material>
     </visual>
@@ -203,5 +188,5 @@
       </geometry>
       <material name="wheel_material">
-        <color rgba="0.0 0.0 0.0 1.0"/>
+        <color rgba="1.0 0.91 0.09 1.0"/>
       </material>
     </visual>
@@ -218,49 +203,22 @@
     </inertial>
   </link>
-  <!-- Camera Stick Link -->
-  <link name="camera_stick_link">
-    <collision>
+  <!-- LiDAR link -->
+  <link name="laser_frame">
+    <visual>
+      <geometry>
+        <cylinder radius="0.065" length="0.078"/>
+      </geometry>
+      <material name="orange">
+        <color rgba="1.00 0.40 0.00 1.00"/>
+      </material>
+    </visual>
+    <collision>
+      <geometry>
+        <cylinder radius="0.065" length="0.078"/>
+      </geometry>
+    </collision>
+    <xacro:inertial_cylinder mass="0.1" length="0.078" radius="0.05">
       <origin xyz="0 0 0" rpy="0 0 0"/>
-      <geometry>
-        <box size="${camera_stick_size} ${camera_stick_size} ${camera_height}"/>
-      </geometry>
-    </collision>
-    <visual>
-      <origin xyz="0 0 0" rpy="0 0 0"/>
-      <geometry>
-        <box size="${camera_stick_size} ${camera_stick_size} ${camera_height}"/>
-      </geometry>
-      <material name="camera_stick_material">
-        <color rgba="0.25 0.25 0.25 1.0"/>
-      </material>
-    </visual>
-    <inertial>
-      <mass value="1e-5" />
-      <origin xyz="0 0 0" rpy="0 0 0"/>
-      <inertia ixx="1e-6" ixy="0" ixz="0" iyy="1e-6" iyz="0" izz="1e-6" />
-    </inertial>
-  </link>
-  <!-- Camera Link -->
-  <link name="camera_link">
-    <collision>
-      <origin xyz="0 0 0" rpy="0 0 0"/>
-      <geometry>
-        <box size="${camera_box_size} ${camera_box_size} ${camera_box_size}"/>
-      </geometry>
-    </collision>
-    <visual>
-      <origin xyz="0 0 0" rpy="0 0 0"/>
-      <geometry>
-        <box size="${camera_box_size} ${camera_box_size} ${camera_box_size}"/>
-      </geometry>
-      <material name="camera_material">
-        <color rgba="0.0 0.0 0.0 1.0"/>
-      </material>
-    </visual>
-    <inertial>
-      <mass value="1e-5" />
-      <origin xyz="0 0 0" rpy="0 0 0"/>
-      <inertia ixx="1e-6" ixy="0" ixz="0" iyy="1e-6" iyz="0" izz="1e-6" />
-    </inertial>
+    </xacro:inertial_cylinder>
   </link>
   <!-- Joints -->
@@ -319,17 +277,9 @@
     <dynamics damping="0.1" friction="0.1"/>
   </joint>
-  <!-- Camera Stick Joint -->
-  <joint name="camera_stick_joint" type="fixed">
-    <axis xyz="0 1 0" />
-    <origin xyz="${body_length/2 - camera_stick_size/2} ${camera_box_size/2 + camera_stick_size/2} ${camera_height/2}" rpy="0.0 0.0 0.0"/>
-    <parent link="body_link"/>
-    <child link="camera_stick_link"/>
-  </joint>
-  <!-- Camera Joint -->
-  <joint name="camera_joint" type="fixed">
-    <axis xyz="0 1 0" />
-    <origin xyz="0.0 ${-camera_box_size/2 - camera_stick_size/2} ${camera_height/2}" rpy="0 ${camera_pitch} 0"/>
-    <parent link="camera_stick_link"/>
-    <child link="camera_link"/>
+  <!-- LiDAR Joint -->
+  <joint name="laser_joint" type="fixed">
+    <parent link="body_link"/>
+    <child link="laser_frame"/>
+    <origin xyz="0.0975 0 0.264" rpy="0 0 0"/>
   </joint>
   <!-- Gazebo Parameters -->
@@ -353,4 +303,27 @@
     <mu1>100.0</mu1>
     <mu2>100.0</mu2>
+  </gazebo>
+  <!-- Sensor Details -->
+  <gazebo reference="laser_frame">
+    <sensor name="laser" type="gpu_lidar">
+      <pose> 0 0 0 0 0 0 0 </pose>
+      <visualize>false</visualize>
+      <update_rate>10</update_rate>
+      <lidar>
+        <scan>
+          <horizontal>
+            <samples>360</samples>
+            <min_angle>-3/14</min_angle>
+            <max_angle>3.14</max_angle>
+          </horizontal>
+        </scan>
+        <range>
+          <min>0.3</min>
+          <max>8.0</max>
+        </range>
+      </lidar>
+      <topic>scan</topic>
+      <gz_frame_id>laser_frame</gz_frame_id>
+    </sensor>
   </gazebo>
   <!-- Gazebo Control -->
@@ -414,40 +387,3 @@
     </plugin>
   </gazebo>
-  <!-- Camera -->
-  <gazebo reference="camera_link">
-    <sensor type="camera" name="vehicle_front_camera">
-      <update_rate>${camera_fps}</update_rate>
-      <visualize>true</visualize>
-      <topic>camera</topic>
-      <camera name="head">
-        <horizontal_fov>${camera_fov}</horizontal_fov>
-        <image>
-          <width>${image_width}</width>
-          <height>${image_height}</height>
-          <format>R8G8B8</format>
-        </image>
-        <clip>
-          <near>0.02</near>
-          <far>300</far>
-        </clip>
-        <noise>
-          <type>gaussian</type>
-          <mean>0.0</mean>
-          <stddev>0.007</stddev>
-        </noise>
-      </camera>
-      <plugin name="camera_controller" filename="libgazebo_ros_camera.so">
-        <alwaysOn>true</alwaysOn>
-        <updateRate>0.0</updateRate>
-        <cameraName>vehicle_front_camera</cameraName>
-        <frameName>camera_link</frameName>
-        <hackBaseline>0.07</hackBaseline>
-        <distortionK1>0.0</distortionK1>
-        <distortionK2>0.0</distortionK2>
-        <distortionK3>0.0</distortionK3>
-        <distortionT1>0.0</distortionT1>
-        <distortionT2>0.0</distortionT2>
-      </plugin>
-    </sensor>
-  </gazebo>
 </robot>
